Commit message: New robots with robotiq gripper and wrist camera

File: mani_skill/assets/robots/panda/panda_v2_gripper_wristcam.urdf (robot description, URDF)
Before this commit: robot panda_gripper, 12 links, 11 joints
Links:
- link camera_link: geometry collision box size=0.02005 0.099 0.023; visual mesh filename=../realsense2_description/meshes/d415.stl

File: mani_skill/assets/robots/panda/panda_v3.urdf (robot description, URDF)
Before this commit: robot panda, 15 links, 14 joints
Links:
- link camera_link: geometry collision box size=0.02005 0.099 0.023; visual mesh filename=../realsense2_description/meshes/d415.stl

File: mani_skill/assets/robots/ur/ur5_pandahand_realsense.urdf (robot description, URDF)
Before this commit: robot ur5, 19 links, 18 joints
Links:
- link camera_link: geometry collision box size=0.02005 0.099 0.023; visual mesh filename=../realsense2_description/meshes/d415.stl
