Commit message: Five new tasks added

File: mani_skill/assets/robots/robotiq_2f/floating_robotiq_2f_85_wristcam.urdf (robot description, URDF)
Before this commit: robot robotiq_arg2f_85_model, 20 links, 19 joints
Joints:
- joint root_x_rot_joint: limit lower=-20 upper=20 effort=100 velocity=0.50 -> lower=-3.15 upper=3.15 effort=100 velocity=0.50
- joint root_y_rot_joint: limit lower=-20 upper=20 effort=100 velocity=0.50 -> lower=-3.15 upper=3.15 effort=100 velocity=0.50
- joint root_z_rot_joint: limit lower=-20 upper=20 effort=100 velocity=0.50 -> lower=-3.15 upper=3.15 effort=100 velocity=0.50

Commit message: HangMug motion planning solver fixed

File: mani_skill/assets/robots/robotiq_2f/floating_robotiq_2f_85_wristcam.urdf (robot description, URDF)
Before this commit: robot robotiq_arg2f_85_model, 20 links, 19 joints
Joints:
- joint root_x_rot_joint: limit lower=-3.15 upper=3.15 effort=100 velocity=0.50 -> lower=-20 upper=20 effort=100 velocity=0.50
- joint root_y_rot_joint: limit lower=-3.15 upper=3.15 effort=100 velocity=0.50 -> lower=-20 upper=20 effort=100 velocity=0.50
- joint root_z_rot_joint: limit lower=-3.15 upper=3.15 effort=100 velocity=0.50 -> lower=-20 upper=20 effort=100 velocity=0.50
